Commit message: Added Simulation Stack

File: dogtooth_description/description/dogtooth_hardware.urdf.xacro (robot description, xacro)
@@ -4,9 +4,9 @@
   <xacro:arg name="prefix" default="" />
   <xacro:arg name="use_mock_hardware" default="false" />
-  <xacro:include filename="$(find dogtooth_base)/description/robot_core.xacro" />
+  <xacro:include filename="$(find dogtooth_description)/description/robot_core.xacro" />
   <!-- Import Rviz colors
   <xacro:include filename="$(find ros2_control_demo_description)/diffbot/urdf/diffbot.materials.xacro" /> -->
   <!-- Import diffbot ros2_control description -->
-  <xacro:include filename="$(find dogtooth_base)/description/dogtooth.ros2_control.xacro" />
+  <xacro:include filename="$(find dogtooth_control)/description/dogtooth.ros2_control.xacro" />
   <xacro:dogbot prefix="$(arg prefix)" />
   <xacro:diffbot_ros2_control

File: dogtooth_description/description/robot_core.xacro (robot description, xacro)
@@ -1,5 +1,5 @@
 <?xml version="1.0"?>
 <robot xmlns:xacro="http://www.ros.org/wiki/xacro" >
- <xacro:macro name="dogbot" params="prefix">
+<xacro:macro name="dogbot" params="prefix">
     <xacro:property name="chassis_xyz" value="-0.016 -0.01 0.1025"/>
     <!-- BASE LINK -->
