Commit message: sensor tf commit

File: dogtooth_description/description/dogtooth.urdf.xacro (robot description, xacro)
@@ -3,7 +3,8 @@
     <xacro:arg name="prefix" default="" />
     <xacro:arg name="use_ros2_control" default="true"/>
+    <xacro:arg name="is_sim" default="true"/>
     <!-- <xacro:include filename="robot_core.xacro"/> -->
     <xacro:include filename="$(find dogtooth_description)/description/dogtooth_core.urdf.xacro"/>
-    <xacro:dogbot prefix="$(arg prefix)" />
+    <xacro:dogbot prefix="$(arg prefix)" is_sim="$(arg is_sim)"/>
     <xacro:if value="$(arg use_ros2_control)">
         <xacro:include filename="$(find dogtooth_description)/description/ros2_control.xacro" />

File: dogtooth_description/description/dogtooth_core.urdf.xacro (robot description, xacro)
@@ -2,5 +2,5 @@
 <robot xmlns:xacro="http://www.ros.org/wiki/xacro" >
 <xacro:include filename="$(find dogtooth_description)/description/wheel.urdf.xacro"/>
-<xacro:macro name="dogbot" params="prefix:=''">
+<xacro:macro name="dogbot" params="prefix:='' is_sim:=true">
      <!-- Base Size -->
     <xacro:property name="base_x_size" value="0.98740000" />
@@ -59,16 +59,8 @@
       <child link="${prefix}inertial_link" />
     </joint>
-    <xacro:dogtooth_wheel wheel_prefix="${prefix}front_left">
-      <origin xyz="${wheelbase/2} ${track/2} ${wheel_vertical_offset}" rpy="0 0 0" />
-    </xacro:dogtooth_wheel>
-    <xacro:dogtooth_wheel wheel_prefix="${prefix}front_right">
-      <origin xyz="${wheelbase/2} ${-track/2} ${wheel_vertical_offset}" rpy="0 0 0" />
-    </xacro:dogtooth_wheel>
-    <xacro:dogtooth_wheel wheel_prefix="${prefix}back_left">
-      <origin xyz="${-wheelbase/2} ${track/2} ${wheel_vertical_offset}" rpy="0 0 0" />
-    </xacro:dogtooth_wheel>
-    <xacro:dogtooth_wheel wheel_prefix="${prefix}back_right">
-      <origin xyz="${-wheelbase/2} ${-track/2} ${wheel_vertical_offset}" rpy="0 0 0" />
-    </xacro:dogtooth_wheel>
+    <xacro:dogtooth_wheel wheel_prefix="${prefix}front_left" x="${wheelbase/2}" y="${track/2}" z="${wheel_vertical_offset}" is_sim="${is_sim}"/>
+    <xacro:dogtooth_wheel wheel_prefix="${prefix}front_right" x="${wheelbase/2}" y="${-track/2}" z="${wheel_vertical_offset}" is_sim="${is_sim}"/>
+    <xacro:dogtooth_wheel wheel_prefix="${prefix}back_left" x="${-wheelbase/2}" y="${track/2}" z="${wheel_vertical_offset}" is_sim="${is_sim}"/>
+    <xacro:dogtooth_wheel wheel_prefix="${prefix}back_right" x="${-wheelbase/2}" y="${-track/2}" z="${wheel_vertical_offset}" is_sim="${is_sim}"/>
 </xacro:macro>
 </robot>

File: dogtooth_description/description/dogtooth_hardware.urdf.xacro (robot description, xacro)
@@ -4,10 +4,12 @@
   <xacro:arg name="prefix" default="" />
   <xacro:arg name="use_mock_hardware" default="false" />
-  <xacro:include filename="$(find dogtooth_description)/description/robot_core.xacro" />
+  <!-- <xacro:include filename="$(find dogtooth_description)/description/robot_core.xacro" /> -->
+  <xacro:include filename="$(find dogtooth_description)/description/dogtooth_core.urdf.xacro"/>
+  <xacro:dogbot prefix="$(arg prefix)" is_sim='false'/>
   <!-- Import Rviz colors
   <xacro:include filename="$(find ros2_control_demo_description)/diffbot/urdf/diffbot.materials.xacro" /> -->
   <!-- Import diffbot ros2_control description -->
   <xacro:include filename="$(find dogtooth_description)/description/dogtooth.ros2_control.xacro" />
-  <xacro:dogbot prefix="$(arg prefix)" />
+  <!-- <xacro:dogbot prefix="$(arg prefix)" /> -->
   <xacro:diffbot_ros2_control
     name="DiffBot" prefix="$(arg prefix)" use_mock_hardware="$(arg use_mock_hardware)"/>

File: dogtooth_description/description/wheel.urdf.xacro (robot description, xacro)
@@ -1,5 +1,5 @@
 <?xml version="1.0"?>
 <robot xmlns:xacro="http://ros.org/wiki/xacro" name="dogtooth_wheel">
-  <xacro:macro name="dogtooth_wheel" params="wheel_prefix *joint_pose">
+  <xacro:macro name="dogtooth_wheel" params="wheel_prefix x y z roll:=0.0 pitch:=0.0 yaw:=0.0 is_sim:=true">
     <link name="${wheel_prefix}_wheel">
       <inertial>
@@ -21,4 +21,11 @@
       </collision>
     </link>
+  <xacro:if value="${is_sim}">
+      <joint name="${wheel_prefix}_wheel_joint" type="continuous">
+      <parent link="base_link"/>
+      <child link="${wheel_prefix}_wheel"/>
+      <origin xyz="${x} ${y} ${z}" rpy="${roll} ${pitch} ${yaw}"/>
+      <axis xyz="0 1 0" rpy="0 0 0" />
+    </joint>
     <gazebo reference="${wheel_prefix}_wheel">
       <mu1 value="1.0"/>
@@ -28,10 +35,13 @@
       <fdir1 value="1 0 0"/>
     </gazebo>
-    <joint name="${wheel_prefix}_wheel_joint" type="continuous">
+  </xacro:if>
+  <xacro:unless value="${is_sim}">
+    <joint name="${wheel_prefix}_wheel_joint" type="fixed">
       <parent link="base_link"/>
       <child link="${wheel_prefix}_wheel"/>
-      <xacro:insert_block name="joint_pose"/>
+      <origin xyz="${x} ${y} ${z}" rpy="${roll} ${pitch} ${yaw}"/>
       <axis xyz="0 1 0" rpy="0 0 0" />
     </joint>
+  </xacro:unless>
   </xacro:macro>
 </robot>
