Commit message: further progress ...

File: hunter_description/description/gazebo_control.xacro (robot description, xacro)
@@ -1,30 +1,44 @@
 <?xml version="1.0"?>
 <robot xmlns:xacro="http://www.ros.org/wiki/xacro">
-<!-- REF: https://github.com/ros-simulation/gazebo_ros_pkgs/wiki/ROS-2-Migration:-Skid-Steer-drive -->
-    <gazebo>
-        <plugin name="skid_steer_drive_controller" filename="libgazebo_ros_diff_drive.so">
-            <update_rate>500</update_rate>
-            <num_wheel_pairs>2</num_wheel_pairs>
-            <!-- FRONT -->
-            <left_joint>front_left_wheel_joint</left_joint>
-            <right_joint>front_right_wheel_joint</right_joint>
-            <!-- REAR -->
-            <left_joint>back_left_wheel_joint</left_joint>
-            <right_joint>back_right_wheel_joint</right_joint>
-            <!-- KINEMATICS -->
-            <wheel_separation>0.525</wheel_separation>
-            <wheel_separation>0.525</wheel_separation>
-            <wheel_diameter>0.279</wheel_diameter>
-            <wheel_diameter>0.279</wheel_diameter>
-            <!-- Limits -->
-            <max_wheel_torque>100</max_wheel_torque>
-            <max_wheel_acceleration>5.0</max_wheel_acceleration>
-            <!-- Output -->
-            <odometry_frame>odom</odometry_frame>
-            <robot_base_frame>base_link</robot_base_frame>
-            <publish_odom>true</publish_odom>
-            <publish_odom_tf>true</publish_odom_tf>
-            <publish_wheel_tf>true</publish_wheel_tf>
-        </plugin>
-    </gazebo>
+  <!-- REF: https://github.com/ros-simulation/gazebo_ros_pkgs/blob/dashing/gazebo_plugins/worlds/gazebo_ros_ackermann_drive_demo.world -->
+  <!-- REF: https://docs.ros.org/en/ros2_packages/rolling/api/gazebo_plugins/generated/classgazebo__plugins_1_1GazeboRosAckermannDrive.html -->
+  <gazebo>
+    <plugin name="gazebo_ros_ackermann_drive" filename="libgazebo_ros_ackermann_drive.so">
+      <ros>
+        <!-- <namespace>demo</namespace> -->
+        <remapping>cmd_vel:=cmd_vel</remapping>
+        <remapping>odom:=odom</remapping>
+        <remapping>distance:=distance</remapping>
+      </ros>
+      <update_rate>100.0</update_rate>
+      <!-- wheels -->
+      <front_left_joint>front_left_wheel_joint</front_left_joint>
+      <front_right_joint>front_right_wheel_joint</front_right_joint>
+      <rear_left_joint>rear_left_wheel_joint</rear_left_joint>
+      <rear_right_joint>rear_right_wheel_joint</rear_right_joint>
+      <left_steering_joint>front_left_steer_joint</left_steering_joint>
+      <right_steering_joint>front_right_steer_joint</right_steering_joint>
+      <steering_wheel_joint>front_steer_joint</steering_wheel_joint>
+      <!-- Max absolute steer angle for tyre in radians-->
+      <!-- Any cmd_vel angular z greater than this would be capped -->
+      <max_steer>0.69</max_steer>
+      <max_steering_angle>7.85</max_steering_angle>
+      <!-- Max absolute linear speed in m/s -->
+      <max_speed>20</max_speed>
+      <!-- PID tuning -->
+      <left_steering_pid_gain>1500 0 1</left_steering_pid_gain>
+      <left_steering_i_range>0 0</left_steering_i_range>
+      <right_steering_pid_gain>1500 0 1</right_steering_pid_gain>
+      <right_steering_i_range>0 0</right_steering_i_range>
+      <linear_velocity_pid_gain>1000 0 1</linear_velocity_pid_gain>
+      <linear_velocity_i_range>0 0</linear_velocity_i_range>
+      <!-- output -->
+      <publish_odom>true</publish_odom>
+      <publish_odom_tf>true</publish_odom_tf>
+      <publish_wheel_tf>true</publish_wheel_tf>
+      <publish_distance>true</publish_distance>
+      <odometry_frame>odom</odometry_frame>
+      <robot_base_frame>base_link</robot_base_frame>
+    </plugin>
+  </gazebo>
 </robot>

File: hunter_description/description/robot.urdf.xacro (robot description, xacro)
@@ -1,10 +1,11 @@
 <?xml version="1.0"?>
 <robot xmlns:xacro="http://www.ros.org/wiki/xacro"  name="robot">
-    <xacro:arg name="prefix" default="" />
     <xacro:arg name="use_ros2_control" default="true"/>
     <xacro:arg name="is_sim" default="true"/>
+    <xacro:include filename="robot_core.xacro" />
+    <xacro:include filename="gazebo_control.xacro" />
     <!-- <xacro:include filename="robot_core.xacro"/> -->
-    <xacro:include filename="$(find hunter_description)/description/hunter_core.urdf.xacro"/>
-    <xacro:dogbot prefix="$(arg prefix)" is_sim="$(arg is_sim)"/>
+    <!-- <xacro:include filename="$(find hunter_description)/description/robot_core.xacro"/>
+    <xacro:hunter_2 prefix="$(arg prefix)" />
     <xacro:if value="$(arg use_ros2_control)">
         <xacro:include filename="$(find hunter_description)/description/ros2_control.xacro" />
@@ -12,4 +13,4 @@
     <xacro:unless value="$(arg use_ros2_control)">
         <xacro:include filename="$(find hunter_description)/description/gazebo_control.xacro" />
-    </xacro:unless>
+    </xacro:unless> -->
 </robot>

File: hunter_description/description/robot_core.xacro (robot description, xacro)
@@ -1,5 +1,4 @@
 <?xml version="1.0"?>
-<robot xmlns:xacro="http://www.ros.org/wiki/xacro" name="robot" >
-    <!-- <xacro:macro name="hunter_2" params="prefix"> -->
+<robot xmlns:xacro="http://www.ros.org/wiki/xacro">
     <!-- REF: https://youtu.be/BcjHyhV0kIs?si=dUpg7IF-kHSUgB-w -->
     <!-- Robot website: https://robosavvy.co.uk/agilex-hunter-2b.html -->
@@ -36,5 +35,6 @@
         <origin xyz="-0.28 0.29249 -0.19558" rpy="${pi/2} 0 0" />
         <axis   xyz="0 0 -1" />
-        <dynamics damping="0.0" friction="15"/>    </joint>
+        <dynamics damping="0.0" friction="15"/>
+    </joint>
     <link name="rear_left_wheel">
         <visual>
@@ -77,6 +77,39 @@
     </link>
     <!-- ============================================================================ -->
+    <!-- FRONT STEER JOINT & LINK -->
+    <joint name="front_steer_joint" type="fixed">
+        <origin xyz="0.44792 -1.1431E-05 -0.121" rpy="0 0 0" />
+        <parent link="chassis" />
+        <child  link="front_steer" />
+        <axis   xyz="0 0 0" />
+    </joint>
+    <link name="front_steer">
+        <visual>
+            <origin xyz="0 0 0" rpy="0 0 0" />
+            <geometry>
+                <mesh filename="file://$(find hunter_description)/meshes/front_steer_link.STL" />
+            </geometry>
+        </visual>
+        <collision>
+            <origin xyz="0 0 0" rpy="0 0 0" />
+            <geometry>
+                <mesh filename="file://$(find hunter_description)/meshes/front_steer_link.STL" />
+            </geometry>
+        </collision>
+        <inertial>
+            <origin xyz="0.049836 8.1046E-15 0.017912" rpy="0 0 0" />
+            <mass value="0.0049179" />
+            <inertia
+                ixx="1.6846E-07"
+                ixy="7.6396E-23"
+                ixz="-1.0974E-08"
+                iyy="7.549E-07"
+                iyz="-1.8957E-22"
+                izz="7.334E-07" />
+        </inertial>
+    </link>
+    <!-- ============================================================================ -->
     <!-- FRONT STEER LEFT WHEEL JOINT & LINK -->
-    <joint name="front_steer_left_wheel_joint" type="revolute">
+    <joint name="front_left_steer_joint" type="revolute">
         <parent link="chassis"/>
         <child link="front_steer_left_wheel"/>
@@ -140,5 +173,5 @@
     <!-- ============================================================================ -->
     <!-- FRONT STEER RIGHT WHEEL JOINT & LINK -->
-    <joint name="front_steer_right_wheel_joint" type="revolute">
+    <joint name="front_right_steer_joint" type="revolute">
         <parent link="chassis"/>
         <child link="front_steer_right_wheel"/>
@@ -200,4 +233,3 @@
         <xacro:inertial_wheel/>
     </link>
-    <!-- </xacro:macro> -->
 </robot>
