Commit message: WIP

File: hunter_description/description/inertial_macros.xacro (robot description, xacro)
@@ -1,36 +1,52 @@
 <?xml version="1.0"?>
 <robot xmlns:xacro="http://www.ros.org/wiki/xacro" >
-    <!-- The values are from: https://github.com/agilexrobotics/ugv_gazebo_sim/blob/master/hunter/hunter2_base/urdf/hunter2_base_gazebo.xacro -->
-    <xacro:macro name="inertial_chassis">
-        <inertial>
-        <origin
-            xyz="0.0266989327622036 0.000409203500587652 -0.135901124750884"
-            rpy="0 0 0" />
-        <mass
-            value="72" />
-        <inertia
-            ixx="0.0332370959804736"
-            ixy="-1.013150489971E-06"
-            ixz="-0.00188859201421112"
-            iyy="0.111072002332437"
-            iyz="-5.13308150598312E-07"
-            izz="0.12660862809283" />
-        </inertial>
-    </xacro:macro>
-    <xacro:macro name="inertial_wheel">
-        <inertial>
-        <origin
-            xyz="-6.5774E-06 2.0242E-05 -0.0096386"
-            rpy="0 0 0" />
-        <mass
-            value="7.0" />
-        <inertia
-            ixx="0.063724"
-            ixy="0"
-            ixz="0"
-            iyy="0.063724"
-            iyz="0"
-            izz="0.11072" />
-        </inertial>
-    </xacro:macro>
+  <!-- The values are from: https://github.com/agilexrobotics/ugv_gazebo_sim/blob/master/hunter/hunter2_base/urdf/hunter2_base_gazebo.xacro -->
+  <xacro:macro name="inertial_chassis">
+    <inertial>
+      <origin
+        xyz="0.0266989327622036 0.000409203500587652 -0.135901124750884"
+        rpy="0 0 0" />
+      <mass
+        value="72" />
+      <inertia
+        ixx="0.0332370959804736"
+        ixy="-1.013150489971E-06"
+        ixz="-0.00188859201421112"
+        iyy="0.111072002332437"
+        iyz="-5.13308150598312E-07"
+        izz="0.12660862809283" />
+    </inertial>
+  </xacro:macro>
+  <xacro:macro name="inertial_wheel">
+    <inertial>
+      <origin
+        xyz="-6.5774E-06 2.0242E-05 -0.0096386"
+        rpy="0 0 0" />
+      <mass
+        value="7.0" />
+      <inertia
+        ixx="0.063724"
+        ixy="0"
+        ixz="0"
+        iyy="0.063724"
+        iyz="0"
+        izz="0.11072" />
+    </inertial>
+  </xacro:macro>
+  <xacro:macro name="inertial_steering_link">
+    <inertial>
+      <origin
+        xyz="0 0 0"
+        rpy="0 0 0" />
+      <mass
+        value="0.005" />
+      <inertia
+        ixx="0.1"
+        ixy="0"
+        ixz="0"
+        iyy="0.1"
+        iyz="0"
+        izz="0.1" />
+    </inertial>
+  </xacro:macro>
 </robot>

File: hunter_description/description/meshes.xacro (robot description, xacro)
@@ -1,17 +1,28 @@
 <?xml version="1.0"?>
 <robot xmlns:xacro="http://www.ros.org/wiki/xacro" >
-    <xacro:macro name="mesh" params="name">
-        <visual>
-            <origin xyz="0 0 0" rpy="0 0 0"/>
-            <geometry>
-                <mesh filename="file://$(find hunter_description)/meshes/${name}.dae" />
-            </geometry>
-        </visual>
-        <collision>
-            <origin xyz="0 0 0" rpy="0 0 0"/>
-            <geometry>
-                <mesh filename="file://$(find hunter_description)/meshes/${name}.dae" />
-            </geometry>
-        </collision>
-    </xacro:macro>
+  <xacro:macro name="mesh" params="name">
+    <visual>
+      <origin xyz="0 0 0" rpy="0 0 0"/>
+      <geometry>
+        <mesh filename="file://$(find hunter_description)/meshes/${name}.dae" />
+      </geometry>
+    </visual>
+    <collision>
+      <origin xyz="0 0 0" rpy="0 0 0"/>
+      <geometry>
+        <mesh filename="file://$(find hunter_description)/meshes/${name}.dae" />
+      </geometry>
+    </collision>
+  </xacro:macro>
+  <xacro:macro name="virtual">
+    <visual>
+      <origin xyz="0 0 0" rpy="0 0 0"/>
+      <geometry>
+        <cylinder length="0.01" radius="0.01"/>
+      </geometry>
+      <material name="invisible">
+        <color rgba="0.0 0.0 0.0 0.0"/>
+      </material>
+    </visual>
+  </xacro:macro>
 </robot>

File: hunter_description/description/robot.urdf.xacro (robot description, xacro)
@@ -1,7 +1,9 @@
 <?xml version="1.0"?>
 <robot xmlns:xacro="http://www.ros.org/wiki/xacro"  name="hunter">
-    <xacro:include filename="robot_core.xacro" />
-    <xacro:include filename="ros2_control.xacro" />
-    <xacro:hunter />
-    <xacro:hunter_ros2_control name="hunter" />
+  <xacro:include filename="$(find hunter_description)/description/robot_core.xacro" />
+  <xacro:include filename="$(find hunter_description)/description/ros2_control.xacro" />
+  <!-- <xacro:include filename="robot_core.xacro" />
+  <xacro:include filename="ros2_control.xacro" /> -->
+  <!-- <xacro:hunter />
+  <xacro:hunter_ros2_control name="hunter" /> -->
 </robot>

File: hunter_description/description/robot_core.xacro (robot description, xacro)
@@ -1,122 +1,105 @@
 <?xml version="1.0"?>
 <robot xmlns:xacro="http://www.ros.org/wiki/xacro">
-    <xacro:macro name="hunter">
-    <!-- REF: https://youtu.be/BcjHyhV0kIs?si=dUpg7IF-kHSUgB-w -->
-    <!-- Robot website: https://robosavvy.co.uk/agilex-hunter-2b.html -->
-    <!-- Include the inertial values from the following -->
-    <xacro:include filename="inertial_macros.xacro"/>
-    <xacro:include filename="meshes.xacro"/>
-    <!-- Constants for robot dimensions -->
-    <xacro:property name="z_base_to_wheel" value="-0.19558" />
-    <xacro:property name="x_base_to_rear" value="-0.28" />
-    <xacro:property name="x_base_to_front" value="0.37142" />
-    <xacro:property name="y_base_to_wheel" value="0.2925" />
-    <xacro:property name="max_steer_angle_central" value="0.461" />
-    <!-- BASE LINK ================================================================== -->
-    <link name="base_link"/>
-    <!-- CHASSIS JOINT & LINK ======================================================= -->
-    <joint name="chassis_joint" type="fixed">
-        <parent link="base_link"/>
-        <child link="chassis"/>
-        <origin xyz="0 0 0.37" rpy="0 0 0" />
-    </joint>
-    <link name="chassis">
-        <xacro:mesh name="chassis"/>
-        <xacro:inertial_chassis/>
-    </link>
-    <!-- REAR WHEELS ================================================================ -->
-    <!-- VIRTUAL REAR WHEEL -->
-    <link name="virtual_rear_wheel"/>
-    <joint name="virtual_rear_wheel_joint" type="continuous">
-        <parent link="chassis"/>
-        <child link="virtual_rear_wheel"/>
-        <origin xyz="${x_base_to_rear} 0.0 ${z_base_to_wheel}" rpy="${pi/2} 0 0"/>
-        <axis xyz="0 0 -1"/>
-        <limit effort="10.0" velocity="10.0"/>
-        <dynamics damping="0.2"/>
-    </joint>
-    <!-- REAR LEFT WHEEL JOINT & LINK -->
-    <link name="rear_left_wheel">
-        <xacro:mesh name="rear_left_wheel"/>
-        <xacro:inertial_wheel/>
-    </link>
-    <joint name="rear_left_wheel_joint" type="continuous">
-        <parent link="chassis"/>
-        <child link="rear_left_wheel"/>
-        <origin xyz="${x_base_to_rear} ${y_base_to_wheel} ${z_base_to_wheel}" rpy="${pi/2} 0 0" />
-        <axis   xyz="0 0 -1" />
-        <dynamics damping="0.2" friction="15"/>
-        <limit effort="10.0" velocity="10.0"/>
-        <mimic joint="virtual_rear_wheel_joint" multiplier="1.0" offset="0.0"/>
-    </joint>
-    <!-- REAR RIGHT WHEEL JOINT & LINK -->
-    <link name="rear_right_wheel">
-        <xacro:mesh name="rear_right_wheel"/>
-        <xacro:inertial_wheel/>
-    </link>
-    <joint name="rear_right_wheel_joint" type="continuous">
-        <parent link="chassis"/>
-        <child link="rear_right_wheel"/>
-        <origin xyz="${x_base_to_rear} -${y_base_to_wheel} ${z_base_to_wheel}" rpy="${pi/2} 0 0" />
-        <axis xyz="0.0 0.0 -1.0"/>
-        <dynamics damping="0.2" friction="15"/>
-        <limit effort="10.0" velocity="10.0"/>
-        <mimic joint="virtual_rear_wheel_joint" multiplier="1.0" offset="0.0"/>
-    </joint>
-    <!-- ============================================================================ -->
-    <!-- VIRTUAL FRONT WHEEL -->
-    <link name="virtual_front_wheel"/>
-    <joint name="virtual_front_wheel_joint" type="revolute">
-        <parent link="chassis"/>
-        <child link="virtual_front_wheel"/>
-        <origin xyz="${x_base_to_front} 0 ${z_base_to_wheel}" rpy="${pi/2} 0 0" />
-        <axis   xyz="0 1 0" />
-        <limit  lower="-${max_steer_angle_central}"  upper="${max_steer_angle_central}"  effort="10.0"  velocity="0" />
-        <dynamics damping="0.2"/>
-    </joint>
-    <!-- FRONT LEFT WHEEL JOINT & LINK -->
-    <link name="front_left_wheel"/>
-    <joint name="front_left_wheel_joint" type="revolute">
-        <parent link="chassis"/>
-        <child link="front_left_wheel"/>
-        <origin xyz="${x_base_to_front} ${y_base_to_wheel} ${z_base_to_wheel}" rpy="${pi/2} 0 0" />
-        <axis   xyz="0 1 0" />
-        <limit  lower="-${max_steer_angle_central}"  upper="${max_steer_angle_central}"  effort="10.0"  velocity="0" />
-        <dynamics damping="0.2"/>
-        <mimic joint="virtual_front_wheel_joint" multiplier="1.0" offset="0.0"/>
-    </joint>
-    <link name="front_left_wheel_cont">
-        <xacro:mesh name="front_left_wheel"/>
-        <xacro:inertial_wheel/>
-    </link>
-    <joint name="front_left_wheel_cont_joint" type="continuous">
-        <parent link="front_left_wheel"/>
-        <child link="front_left_wheel_cont"/>
-        <origin xyz="0 0 0" rpy="0 0 0" />
-        <axis   xyz="0 0 -1" />
-        <mimic joint="virtual_rear_wheel_joint" multiplier="1.0" offset="0.0"/>
-    </joint>
-    <!-- FRONT RIGHT WHEEL JOINT & LINK -->
-    <link name="front_right_wheel"/>
-    <joint name="front_right_wheel_joint" type="revolute">
-        <parent link="chassis"/>
-        <child link="front_right_wheel"/>
-        <origin xyz="${x_base_to_front}  -${y_base_to_wheel} ${z_base_to_wheel}" rpy="${pi/2} 0 0" />
-        <axis   xyz="0 1 0" />
-        <limit  lower="-${max_steer_angle_central}"  upper="${max_steer_angle_central}"  effort="10.0"  velocity="0" />
-        <dynamics damping="0.2"/>
-        <mimic joint="virtual_front_wheel_joint" multiplier="1.0" offset="0.0"/>
-    </joint>
-    <link name="front_right_wheel_cont">
-        <xacro:mesh name="front_right_wheel"/>
-        <xacro:inertial_wheel/>
-    </link>
-    <joint name="front_right_wheel_cont_joint" type="continuous">
-        <parent link="front_right_wheel"/>
-        <child link="front_right_wheel_cont"/>
-        <origin xyz="0 0 0" rpy="0 0 0" />
-        <axis   xyz="0 0 -1" />
-        <mimic joint="virtual_rear_wheel_joint" multiplier="1.0" offset="0.0"/>
-    </joint>
-    </xacro:macro>
+  <!-- REF: https://youtu.be/BcjHyhV0kIs?si=dUpg7IF-kHSUgB-w -->
+  <!-- Robot website: https://robosavvy.co.uk/agilex-hunter-2b.html -->
+  <!-- Include the inertial values from the following -->
+  <xacro:include filename="inertial_macros.xacro"/>
+  <xacro:include filename="meshes.xacro"/>
+  <!-- Constants for robot dimensions -->
+  <xacro:property name="z_base_to_wheel" value="-0.19558" />
+  <xacro:property name="x_base_to_rear" value="-0.28" />
+  <xacro:property name="x_base_to_front" value="0.37142" />
+  <xacro:property name="y_base_to_wheel" value="0.2925" />
+  <xacro:property name="max_steer_angle_central" value="0.461" />
+  <!-- BASE LINK ================================================================== -->
+  <link name="base_link"/>
+  <!-- CHASSIS JOINT & LINK ======================================================= -->
+  <joint name="chassis_joint" type="fixed">
+    <parent link="base_link"/>
+    <child link="chassis"/>
+    <origin xyz="0 0 0.37" rpy="0 0 0" />
+  </joint>
+  <link name="chassis">
+    <xacro:mesh name="chassis"/>
+    <xacro:inertial_chassis/>
+  </link>
+  <!-- REAR WHEELS ================================================================ -->
+  <!-- REAR LEFT WHEEL JOINT & LINK -->
+  <link name="rear_left_wheel">
+    <xacro:mesh name="rear_left_wheel"/>
+    <xacro:inertial_wheel/>
+  </link>
+  <joint name="rear_left_wheel_joint" type="continuous">
+    <parent link="chassis"/>
+    <child link="rear_left_wheel"/>
+    <origin xyz="${x_base_to_rear} ${y_base_to_wheel} ${z_base_to_wheel}" rpy="${pi/2} 0 0" />
+    <axis   xyz="0 0 -1" />
+    <dynamics damping="0.2" friction="15"/>
+    <limit effort="10.0" velocity="10.0"/>
+  </joint>
+  <!-- REAR RIGHT WHEEL JOINT & LINK -->
+  <link name="rear_right_wheel">
+    <xacro:mesh name="rear_right_wheel"/>
+    <xacro:inertial_wheel/>
+  </link>
+  <joint name="rear_right_wheel_joint" type="continuous">
+    <parent link="chassis"/>
+    <child link="rear_right_wheel"/>
+    <origin xyz="${x_base_to_rear} -${y_base_to_wheel} ${z_base_to_wheel}" rpy="${pi/2} 0 0" />
+    <axis xyz="0.0 0.0 -1.0"/>
+    <dynamics damping="0.2" friction="15"/>
+    <limit effort="10.0" velocity="10.0"/>
+  </joint>
+  <!-- ============================================================================ -->
+  <!-- FRONT LEFT STEERING JOINT & LINK -->
+  <link name="front_left_steering_link">
+    <xacro:virtual/>
+    <xacro:inertial_steering_link/>
+  </link>
+  <joint name="front_left_steering_joint" type="revolute">
+    <parent link="chassis"/>
+    <child link="front_left_steering_link"/>
+    <origin xyz="${x_base_to_front} ${y_base_to_wheel} ${z_base_to_wheel}" rpy="${pi/2} 0 0" />
+    <axis   xyz="0 1 0" />
+    <limit  lower="-${max_steer_angle_central}"  upper="${max_steer_angle_central}"  effort="10.0"  velocity="0" />
+    <dynamics damping="0.2"/>
+    <!-- <mimic joint="virtual_front_wheel_joint" multiplier="1.0" offset="0.0"/> -->
+  </joint>
+  <!-- FRONT LEFT WHEEL JOINT & LINK -->
+  <link name="front_left_wheel">
+    <xacro:mesh name="front_left_wheel"/>
+    <xacro:inertial_wheel/>
+  </link>
+  <joint name="front_left_wheel_joint" type="continuous">
+    <parent link="front_left_steering_link"/>
+    <child link="front_left_wheel"/>
+    <origin xyz="0 0 0" rpy="0 0 0" />
+    <axis   xyz="0 0 -1" />
+  </joint>
+  <!-- FRONT RIGHT STEERING JOINT & LINK -->
+  <link name="front_right_steering_link">
+    <xacro:virtual/>
+    <xacro:inertial_steering_link/>
+  </link>
+  <joint name="front_right_steering_joint" type="revolute">
+    <parent link="chassis"/>
+    <child link="front_right_steering_link"/>
+    <origin xyz="${x_base_to_front}  -${y_base_to_wheel} ${z_base_to_wheel}" rpy="${pi/2} 0 0" />
+    <axis   xyz="0 1 0" />
+    <limit  lower="-${max_steer_angle_central}"  upper="${max_steer_angle_central}"  effort="10.0"  velocity="0" />
+    <dynamics damping="0.2"/>
+    <!-- <mimic joint="front_left_wheel_joint" multiplier="1.0" offset="0.0"/> -->
+  </joint>
+  <!-- FRONT RIGHT WHEEL JOINT & LINK -->
+  <link name="front_right_wheel">
+    <xacro:mesh name="front_right_wheel"/>
+    <xacro:inertial_wheel/>
+  </link>
+  <joint name="front_right_wheel_joint" type="continuous">
+    <parent link="front_right_steering_link"/>
+    <child link="front_right_wheel"/>
+    <origin xyz="0 0 0" rpy="0 0 0" />
+    <axis   xyz="0 0 -1" />
+    <!-- <mimic joint="rear_left_wheel_joint" multiplier="1.0" offset="0.0"/> -->
+  </joint>
 </robot>

File: hunter_description/description/ros2_control.xacro (robot description, xacro)
@@ -1,19 +1,41 @@
 <?xml version="1.0"?>
 <robot xmlns:xacro="http://www.ros.org/wiki/xacro">
-  <xacro:macro name="hunter_ros2_control" params="name">
-    <ros2_control name="${name}" type="system">
-      <hardware>
-        <plugin>hunter_description/CarlikeBotSystemHardware</plugin>
-      </hardware>
-      <joint name="virtual_front_wheel_joint">
-        <command_interface name="position"/>
-        <state_interface name="position"/>
-      </joint>
-      <joint name="virtual_rear_wheel_joint">
-        <command_interface name="velocity"/>
-        <state_interface name="velocity"/>
-        <state_interface name="position"/>
-      </joint>
-    </ros2_control>
-  </xacro:macro>
+  <ros2_control name="GazeboSystem" type="system">
+    <hardware>
+      <plugin>gazebo_ros2_control/GazeboSystem</plugin>
+    </hardware>
+    <joint name="front_left_steering_joint">
+      <command_interface name="position"/>
+      <state_interface name="position"/>
+    </joint>
+    <joint name="front_right_steering_joint">
+      <command_interface name="position"/>
+      <state_interface name="position"/>
+    </joint>
+    <joint name="front_right_wheel_joint">
+      <!-- <command_interface name="velocity"/> -->
+      <state_interface name="velocity"/>
+      <state_interface name="position"/>
+    </joint>
+    <joint name="front_left_wheel_joint">
+      <!-- <command_interface name="velocity"/> -->
+      <state_interface name="velocity"/>
+      <state_interface name="position"/>
+    </joint>
+    <joint name="rear_right_wheel_joint">
+      <command_interface name="velocity"/>
+      <state_interface name="velocity"/>
+      <state_interface name="position"/>
+    </joint>
+    <joint name="rear_left_wheel_joint">
+      <command_interface name="velocity"/>
+      <state_interface name="velocity"/>
+      <state_interface name="position"/>
+    </joint>
+  </ros2_control>
+  <gazebo>
+    <plugin filename="libgazebo_ros2_control.so" name="gazebo_ros2_control">
+      <parameters>/home/ibrahim/aoc/hunter/install/hunter_description/share/hunter_description/config/ackermann_controller.yaml</parameters>
+    </plugin>
+  </gazebo>
 </robot>

Commit message: WIP - 2

File: hunter_description/description/inertial_macros.xacro (robot description, xacro)
@@ -1,5 +1,4 @@
 <?xml version="1.0"?>
 <robot xmlns:xacro="http://www.ros.org/wiki/xacro" >
-  <!-- The values are from: https://github.com/agilexrobotics/ugv_gazebo_sim/blob/master/hunter/hunter2_base/urdf/hunter2_base_gazebo.xacro -->
   <xacro:macro name="inertial_chassis">
     <inertial>

File: hunter_description/description/robot.urdf.xacro (robot description, xacro)
@@ -1,9 +1,5 @@
 <?xml version="1.0"?>
 <robot xmlns:xacro="http://www.ros.org/wiki/xacro"  name="hunter">
-  <xacro:include filename="$(find hunter_description)/description/robot_core.xacro" />
-  <xacro:include filename="$(find hunter_description)/description/ros2_control.xacro" />
-  <!-- <xacro:include filename="robot_core.xacro" />
-  <xacro:include filename="ros2_control.xacro" /> -->
-  <!-- <xacro:hunter />
-  <xacro:hunter_ros2_control name="hunter" /> -->
+  <xacro:include filename="robot_core.xacro" />
+  <xacro:include filename="ros2_control.xacro" />
 </robot>

File: hunter_description/description/robot_core.xacro (robot description, xacro)
@@ -1,6 +1,4 @@
 <?xml version="1.0"?>
 <robot xmlns:xacro="http://www.ros.org/wiki/xacro">
-  <!-- REF: https://youtu.be/BcjHyhV0kIs?si=dUpg7IF-kHSUgB-w -->
-  <!-- Robot website: https://robosavvy.co.uk/agilex-hunter-2b.html -->
   <!-- Include the inertial values from the following -->
   <xacro:include filename="inertial_macros.xacro"/>
@@ -12,11 +10,9 @@
   <xacro:property name="y_base_to_wheel" value="0.2925" />
   <xacro:property name="max_steer_angle_central" value="0.461" />
-  <!-- BASE LINK ================================================================== -->
   <link name="base_link"/>
-  <!-- CHASSIS JOINT & LINK ======================================================= -->
   <joint name="chassis_joint" type="fixed">
     <parent link="base_link"/>
     <child link="chassis"/>
-    <origin xyz="0 0 0.37" rpy="0 0 0" />
+    <origin rpy="0 0 0" xyz="0 0 0.37"/>
   </joint>
   <link name="chassis">
@@ -24,6 +20,4 @@
     <xacro:inertial_chassis/>
   </link>
-  <!-- REAR WHEELS ================================================================ -->
-  <!-- REAR LEFT WHEEL JOINT & LINK -->
   <link name="rear_left_wheel">
     <xacro:mesh name="rear_left_wheel"/>
@@ -38,5 +32,4 @@
     <limit effort="10.0" velocity="10.0"/>
   </joint>
-  <!-- REAR RIGHT WHEEL JOINT & LINK -->
   <link name="rear_right_wheel">
     <xacro:mesh name="rear_right_wheel"/>
@@ -51,6 +44,4 @@
     <limit effort="10.0" velocity="10.0"/>
   </joint>
-  <!-- ============================================================================ -->
-  <!-- FRONT LEFT STEERING JOINT & LINK -->
   <link name="front_left_steering_link">
     <xacro:virtual/>
@@ -62,9 +53,7 @@
     <origin xyz="${x_base_to_front} ${y_base_to_wheel} ${z_base_to_wheel}" rpy="${pi/2} 0 0" />
     <axis   xyz="0 1 0" />
-    <limit  lower="-${max_steer_angle_central}"  upper="${max_steer_angle_central}"  effort="10.0"  velocity="0" />
+    <limit  lower="-${max_steer_angle_central}"  upper="${max_steer_angle_central}"  effort="10.0"  velocity="1" />
     <dynamics damping="0.2"/>
-    <!-- <mimic joint="virtual_front_wheel_joint" multiplier="1.0" offset="0.0"/> -->
   </joint>
-  <!-- FRONT LEFT WHEEL JOINT & LINK -->
   <link name="front_left_wheel">
     <xacro:mesh name="front_left_wheel"/>
@@ -77,5 +66,4 @@
     <axis   xyz="0 0 -1" />
   </joint>
-  <!-- FRONT RIGHT STEERING JOINT & LINK -->
   <link name="front_right_steering_link">
     <xacro:virtual/>
@@ -87,9 +75,7 @@
     <origin xyz="${x_base_to_front}  -${y_base_to_wheel} ${z_base_to_wheel}" rpy="${pi/2} 0 0" />
     <axis   xyz="0 1 0" />
-    <limit  lower="-${max_steer_angle_central}"  upper="${max_steer_angle_central}"  effort="10.0"  velocity="0" />
+    <limit  lower="-${max_steer_angle_central}"  upper="${max_steer_angle_central}"  effort="10.0"  velocity="1" />
     <dynamics damping="0.2"/>
-    <!-- <mimic joint="front_left_wheel_joint" multiplier="1.0" offset="0.0"/> -->
   </joint>
-  <!-- FRONT RIGHT WHEEL JOINT & LINK -->
   <link name="front_right_wheel">
     <xacro:mesh name="front_right_wheel"/>
@@ -101,5 +87,4 @@
     <origin xyz="0 0 0" rpy="0 0 0" />
     <axis   xyz="0 0 -1" />
-    <!-- <mimic joint="rear_left_wheel_joint" multiplier="1.0" offset="0.0"/> -->
   </joint>
 </robot>
