Commit message: convert to car like robot

File: hunter_description/description/robot.urdf.xacro (robot description, xacro)
@@ -1,16 +1,8 @@
 <?xml version="1.0"?>
-<robot xmlns:xacro="http://www.ros.org/wiki/xacro"  name="robot">
-    <xacro:arg name="use_ros2_control" default="true"/>
+<robot xmlns:xacro="http://www.ros.org/wiki/xacro"  name="hunter">
     <xacro:arg name="is_sim" default="true"/>
     <xacro:include filename="robot_core.xacro" />
-    <xacro:include filename="gazebo_control.xacro" />
-    <!-- <xacro:include filename="robot_core.xacro"/> -->
-    <!-- <xacro:include filename="$(find hunter_description)/description/robot_core.xacro"/>
-    <xacro:hunter_2 prefix="$(arg prefix)" />
-    <xacro:if value="$(arg use_ros2_control)">
-        <xacro:include filename="$(find hunter_description)/description/ros2_control.xacro" />
-    </xacro:if>
-    <xacro:unless value="$(arg use_ros2_control)">
-        <xacro:include filename="$(find hunter_description)/description/gazebo_control.xacro" />
-    </xacro:unless> -->
+    <xacro:include filename="ros2_control.xacro" />
+    <!-- <xacro:carlikebot /> -->
+    <xacro:carlikebot_ros2_control name="CarlikeBot" />
 </robot>

File: hunter_description/description/robot_core.xacro (robot description, xacro)
@@ -5,4 +5,9 @@
     <!-- Include the inertial values from the following -->
     <xacro:include filename="inertial_macros.xacro"/>
+    <!-- Constants for robot dimensions -->
+    <xacro:property name="z_base_to_wheel" value="-0.19558" />
+    <xacro:property name="x_base_to_rear" value="-0.28" />
+    <xacro:property name="x_base_to_front" value="0.37142" />
+    <xacro:property name="y_base_to_wheel" value="0.2925" />
     <!-- BASE LINK ================================================================== -->
     <link name="base_link"/>
@@ -11,5 +16,5 @@
         <parent link="base_link"/>
         <child link="chassis"/>
-        <origin xyz="0 0 0.26" rpy="0 0 0" />
+        <origin xyz="0 0 0.37" rpy="0 0 0" />
     </joint>
     <link name="chassis">
@@ -34,5 +39,5 @@
             <origin xyz="0 0 0" rpy="0 0 0"/>
             <geometry>
-                <cylinder length="0.01" radius="0.165"/>
+                <cylinder length="0.01" radius="0.01"/>
             </geometry>
             <material name="invisible">
@@ -44,5 +49,5 @@
         <parent link="chassis"/>
         <child link="virtual_rear_wheel"/>
-        <origin xyz="-0.28 0.0 -0.19558" rpy="${pi/2} 0 0"/>
+        <origin xyz="${x_base_to_rear} 0.0 ${z_base_to_wheel}" rpy="${pi/2} 0 0"/>
         <axis xyz="0 0 -1"/>
         <limit effort="10.0" velocity="10.0"/>
@@ -68,5 +73,5 @@
         <parent link="chassis"/>
         <child link="rear_left_wheel"/>
-        <origin xyz="-0.28 0.29249 -0.19558" rpy="${pi/2} 0 0" />
+        <origin xyz="${x_base_to_rear} ${y_base_to_wheel} ${z_base_to_wheel}" rpy="${pi/2} 0 0" />
         <axis   xyz="0 0 -1" />
         <dynamics damping="0.2" friction="15"/>
@@ -93,5 +98,5 @@
         <parent link="chassis"/>
         <child link="rear_right_wheel"/>
-        <origin xyz="-0.28018 -0.29251 -0.19558" rpy="${pi/2} 0 0" />
+        <origin xyz="${x_base_to_rear} -${y_base_to_wheel} ${z_base_to_wheel}" rpy="${pi/2} 0 0" />
         <axis xyz="0.0 0.0 -1.0"/>
         <dynamics damping="0.2" friction="15"/>
@@ -105,5 +110,5 @@
             <origin xyz="0 0 0" rpy="0 0 0"/>
             <geometry>
-                <cylinder length="0.01" radius="0.165"/>
+                <cylinder length="0.01" radius="0.01"/>
             </geometry>
             <material name="invisible">
@@ -115,5 +120,5 @@
         <parent link="chassis"/>
         <child link="virtual_front_wheel"/>
-        <origin xyz="0.37142 0 -0.1955" rpy="${pi/2} 0 0" />
+        <origin xyz="${x_base_to_front} 0 ${z_base_to_wheel}" rpy="${pi/2} 0 0" />
         <axis   xyz="0 1 0" />
         <limit  lower="-0.69"  upper="0.69"  effort="10.0"  velocity="0" />
@@ -139,5 +144,5 @@
         <parent link="chassis"/>
         <child link="front_left_wheel"/>
-        <origin xyz="0.37142 0.29199 -0.1955" rpy="${pi/2} 0 0" />
+        <origin xyz="${x_base_to_front} ${y_base_to_wheel} ${z_base_to_wheel}" rpy="${pi/2} 0 0" />
         <axis   xyz="0 1 0" />
         <limit  lower="-0.69"  upper="0.69"  effort="10.0"  velocity="0" />
@@ -164,5 +169,5 @@
         <parent link="chassis"/>
         <child link="front_right_wheel"/>
-        <origin xyz="0.37142 -0.29199 -0.1955" rpy="${pi/2} 0 0" />
+        <origin xyz="${x_base_to_front}  -${y_base_to_wheel} ${z_base_to_wheel}" rpy="${pi/2} 0 0" />
         <axis   xyz="0 1 0" />
         <limit  lower="-0.69"  upper="0.69"  effort="10.0"  velocity="0" />

Commit message: fix steering

File: hunter_description/description/robot.urdf.xacro (robot description, xacro)
@@ -2,4 +2,4 @@
 <robot xmlns:xacro="http://www.ros.org/wiki/xacro"  name="hunter">
   <xacro:include filename="robot_core.xacro" />
-  <xacro:include filename="ros2_control.xacro" />
+  <xacro:include filename="ros2_control_bicycle.xacro" />
 </robot>

File: hunter_description/description/robot_core.xacro (robot description, xacro)
@@ -28,5 +28,5 @@
     <child link="rear_left_wheel"/>
     <origin xyz="${x_base_to_rear} ${y_base_to_wheel} ${z_base_to_wheel}" rpy="${pi/2} 0 0" />
-    <axis   xyz="0 0 -1" />
+    <axis xyz="0 0 -1" />
     <dynamics damping="0.2" friction="15"/>
     <limit effort="10.0" velocity="10.0"/>
@@ -40,7 +40,8 @@
     <child link="rear_right_wheel"/>
     <origin xyz="${x_base_to_rear} -${y_base_to_wheel} ${z_base_to_wheel}" rpy="${pi/2} 0 0" />
-    <axis xyz="0.0 0.0 -1.0"/>
+    <axis xyz="0 0 -1"/>
     <dynamics damping="0.2" friction="15"/>
     <limit effort="10.0" velocity="10.0"/>
+    <mimic joint="rear_left_wheel_joint" multiplier="1.0" offset="0.0"/>
   </joint>
   <link name="front_left_steering_link">
@@ -77,4 +78,5 @@
     <limit  lower="-${max_steer_angle_central}"  upper="${max_steer_angle_central}"  effort="10.0"  velocity="1" />
     <dynamics damping="0.2"/>
+    <mimic joint="front_left_steering_joint" multiplier="1.0" offset="0.0"/>
   </joint>
   <link name="front_right_wheel">
@@ -83,4 +85,5 @@
   </link>
   <joint name="front_right_wheel_joint" type="continuous">
+    <!-- <mimic joint="front_left_wheel_joint"/> -->
     <parent link="front_right_steering_link"/>
     <child link="front_right_wheel"/>

File: hunter_description/description/ros2_control_bicycle.xacro (robot description, xacro)
@@ -10,4 +10,6 @@
     </joint>
     <joint name="front_right_steering_joint">
+      <param name="mimic">front_left_steering_joint</param>
+      <!-- <param name="multiplier">1</param> -->
       <command_interface name="position"/>
       <state_interface name="position"/>
@@ -23,11 +25,13 @@
       <state_interface name="position"/>
     </joint>
-    <joint name="rear_right_wheel_joint">
+    <joint name="rear_left_wheel_joint">
       <command_interface name="velocity"/>
       <state_interface name="velocity"/>
       <state_interface name="position"/>
     </joint>
-    <joint name="rear_left_wheel_joint">
-      <command_interface name="velocity"/>
+    <joint name="rear_right_wheel_joint">
+      <param name="mimic">rear_left_wheel_joint</param>
+      <param name="multiplier">1</param>
+      <!-- <command_interface name="velocity"/> -->
       <state_interface name="velocity"/>
       <state_interface name="position"/>
@@ -36,5 +40,5 @@
   <gazebo>
     <plugin filename="libgazebo_ros2_control.so" name="gazebo_ros2_control">
-      <parameters>/home/ibrahim/aoc/hunter/install/hunter_description/share/hunter_description/config/ackermann_controller.yaml</parameters>
+      <parameters>$(find hunter_description)/config/bicycle_controller.yaml</parameters>
     </plugin>
   </gazebo>

Commit message: clean up

File: hunter_description/description/robot.urdf.xacro (robot description, xacro)
@@ -2,4 +2,4 @@
 <robot xmlns:xacro="http://www.ros.org/wiki/xacro"  name="hunter">
   <xacro:include filename="robot_core.xacro" />
-  <xacro:include filename="ros2_control_bicycle.xacro" />
+  <xacro:include filename="ros2_control.xacro" />
 </robot>

File: hunter_description/description/robot_core.xacro (robot description, xacro)
@@ -85,5 +85,4 @@
   </link>
   <joint name="front_right_wheel_joint" type="continuous">
-    <!-- <mimic joint="front_left_wheel_joint"/> -->
     <parent link="front_right_steering_link"/>
     <child link="front_right_wheel"/>

File: hunter_description/description/ros2_control.xacro (robot description, xacro)
@@ -11,16 +11,5 @@
     <joint name="front_right_steering_joint">
       <param name="mimic">front_left_steering_joint</param>
-      <!-- <param name="multiplier">1</param> -->
-      <command_interface name="position"/>
-      <state_interface name="position"/>
-    </joint>
-    <joint name="front_right_wheel_joint">
-      <!-- <command_interface name="velocity"/> -->
-      <state_interface name="velocity"/>
-      <state_interface name="position"/>
-    </joint>
-    <joint name="front_left_wheel_joint">
-      <!-- <command_interface name="velocity"/> -->
-      <state_interface name="velocity"/>
+      <param name="multiplier">1</param>
       <state_interface name="position"/>
     </joint>
@@ -33,5 +22,12 @@
       <param name="mimic">rear_left_wheel_joint</param>
       <param name="multiplier">1</param>
-      <!-- <command_interface name="velocity"/> -->
+      <state_interface name="velocity"/>
+      <state_interface name="position"/>
+    </joint>
+    <joint name="front_right_wheel_joint">
+      <state_interface name="velocity"/>
+      <state_interface name="position"/>
+    </joint>
+    <joint name="front_left_wheel_joint">
       <state_interface name="velocity"/>
       <state_interface name="position"/>
@@ -40,5 +36,5 @@
   <gazebo>
     <plugin filename="libgazebo_ros2_control.so" name="gazebo_ros2_control">
-      <parameters>$(find hunter_description)/config/bicycle_controller.yaml</parameters>
+      <parameters>$(find hunter_description)/config/ackermann_like_controller.yaml</parameters>
     </plugin>
   </gazebo>
