Commit message: refactor

File: hunter_description/description/meshes.xacro (robot description, xacro)
@@ -1,9 +1,9 @@
 <?xml version="1.0"?>
 <robot xmlns:xacro="http://www.ros.org/wiki/xacro" >
-    <xacro:macro name="chassis_mesh">
+    <xacro:macro name="mesh" params="name">
         <visual>
             <origin xyz="0 0 0" rpy="0 0 0"/>
             <geometry>
-                <mesh filename="file://$(find hunter_description)/meshes/chassis.dae" />
+                <mesh filename="file://$(find hunter_description)/meshes/${name}.dae" />
             </geometry>
         </visual>
@@ -11,61 +11,5 @@
             <origin xyz="0 0 0" rpy="0 0 0"/>
             <geometry>
-                <mesh filename="file://$(find hunter_description)/meshes/chassis.dae" />
-            </geometry>
-        </collision>
-    </xacro:macro>
-    <xacro:macro name="rear_left_wheel_mesh">
-        <visual>
-            <origin xyz="0 0 0" rpy="0 0 0" />
-            <geometry>
-                <mesh filename="file://$(find hunter_description)/meshes/rear_left_wheel.dae" />
-            </geometry>
-        </visual>
-        <collision>
-            <origin xyz="0 0 0" rpy="0 0 0" />
-            <geometry>
-                <mesh filename="file://$(find hunter_description)/meshes/rear_left_wheel.dae" />
-            </geometry>
-        </collision>
-    </xacro:macro>
-    <xacro:macro name="rear_right_wheel_mesh">
-        <visual>
-            <origin xyz="0 0 0" rpy="0 0 0" />
-            <geometry>
-                <mesh filename="file://$(find hunter_description)/meshes/rear_right_wheel.dae" />
-            </geometry>
-        </visual>
-        <collision>
-            <origin xyz="0 0 0" rpy="0 0 0" />
-            <geometry>
-                <mesh filename="file://$(find hunter_description)/meshes/rear_right_wheel.dae" />
-            </geometry>
-        </collision>
-    </xacro:macro>
-    <xacro:macro name="front_left_wheel_mesh">
-        <visual>
-            <origin xyz="0 0 0" rpy="0 0 0" />
-            <geometry>
-                <mesh filename="file://$(find hunter_description)/meshes/front_left_wheel.dae" />
-            </geometry>
-        </visual>
-        <collision>
-            <origin xyz="0 0 0" rpy="0 0 0" />
-            <geometry>
-                <mesh filename="file://$(find hunter_description)/meshes/front_left_wheel.dae" />
-            </geometry>
-        </collision>
-    </xacro:macro>
-    <xacro:macro name="front_right_wheel_mesh">
-        <visual>
-            <origin xyz="0 0 0" rpy="0 0 0" />
-            <geometry>
-                <mesh filename="file://$(find hunter_description)/meshes/front_right_wheel.dae" />
-            </geometry>
-        </visual>
-        <collision>
-            <origin xyz="0 0 0" rpy="0 0 0" />
-            <geometry>
-                <mesh filename="file://$(find hunter_description)/meshes/front_right_wheel.dae" />
+                <mesh filename="file://$(find hunter_description)/meshes/${name}.dae" />
             </geometry>
         </collision>

File: hunter_description/description/robot.urdf.xacro (robot description, xacro)
@@ -1,8 +1,7 @@
 <?xml version="1.0"?>
 <robot xmlns:xacro="http://www.ros.org/wiki/xacro"  name="hunter">
-    <xacro:arg name="is_sim" default="true"/>
     <xacro:include filename="robot_core.xacro" />
     <xacro:include filename="ros2_control.xacro" />
-    <!-- <xacro:carlikebot /> -->
-    <xacro:carlikebot_ros2_control name="CarlikeBot" />
+    <xacro:hunter />
+    <xacro:hunter_ros2_control name="hunter" />
 </robot>

File: hunter_description/description/robot_core.xacro (robot description, xacro)
@@ -1,4 +1,5 @@
 <?xml version="1.0"?>
 <robot xmlns:xacro="http://www.ros.org/wiki/xacro">
+    <xacro:macro name="hunter">
     <!-- REF: https://youtu.be/BcjHyhV0kIs?si=dUpg7IF-kHSUgB-w -->
     <!-- Robot website: https://robosavvy.co.uk/agilex-hunter-2b.html -->
@@ -11,4 +12,5 @@
     <xacro:property name="x_base_to_front" value="0.37142" />
     <xacro:property name="y_base_to_wheel" value="0.2925" />
+    <xacro:property name="max_steer_angle_central" value="0.461" />
     <!-- BASE LINK ================================================================== -->
     <link name="base_link"/>
@@ -20,5 +22,5 @@
     </joint>
     <link name="chassis">
-        <xacro:chassis_mesh/>
+        <xacro:mesh name="chassis"/>
         <xacro:inertial_chassis/>
     </link>
@@ -36,5 +38,5 @@
     <!-- REAR LEFT WHEEL JOINT & LINK -->
     <link name="rear_left_wheel">
-        <xacro:rear_left_wheel_mesh/>
+        <xacro:mesh name="rear_left_wheel"/>
         <xacro:inertial_wheel/>
     </link>
@@ -50,5 +52,5 @@
     <!-- REAR RIGHT WHEEL JOINT & LINK -->
     <link name="rear_right_wheel">
-        <xacro:rear_right_wheel_mesh/>
+        <xacro:mesh name="rear_right_wheel"/>
         <xacro:inertial_wheel/>
     </link>
@@ -70,5 +72,5 @@
         <origin xyz="${x_base_to_front} 0 ${z_base_to_wheel}" rpy="${pi/2} 0 0" />
         <axis   xyz="0 1 0" />
-        <limit  lower="-0.69"  upper="0.69"  effort="10.0"  velocity="0" />
+        <limit  lower="-${max_steer_angle_central}"  upper="${max_steer_angle_central}"  effort="10.0"  velocity="0" />
         <dynamics damping="0.2"/>
     </joint>
@@ -80,10 +82,10 @@
         <origin xyz="${x_base_to_front} ${y_base_to_wheel} ${z_base_to_wheel}" rpy="${pi/2} 0 0" />
         <axis   xyz="0 1 0" />
-        <limit  lower="-0.69"  upper="0.69"  effort="10.0"  velocity="0" />
+        <limit  lower="-${max_steer_angle_central}"  upper="${max_steer_angle_central}"  effort="10.0"  velocity="0" />
         <dynamics damping="0.2"/>
         <mimic joint="virtual_front_wheel_joint" multiplier="1.0" offset="0.0"/>
     </joint>
     <link name="front_left_wheel_cont">
-        <xacro:front_left_wheel_mesh/>
+        <xacro:mesh name="front_left_wheel"/>
         <xacro:inertial_wheel/>
     </link>
@@ -102,10 +104,10 @@
         <origin xyz="${x_base_to_front}  -${y_base_to_wheel} ${z_base_to_wheel}" rpy="${pi/2} 0 0" />
         <axis   xyz="0 1 0" />
-        <limit  lower="-0.69"  upper="0.69"  effort="10.0"  velocity="0" />
+        <limit  lower="-${max_steer_angle_central}"  upper="${max_steer_angle_central}"  effort="10.0"  velocity="0" />
         <dynamics damping="0.2"/>
         <mimic joint="virtual_front_wheel_joint" multiplier="1.0" offset="0.0"/>
     </joint>
     <link name="front_right_wheel_cont">
-        <xacro:front_right_wheel_mesh/>
+        <xacro:mesh name="front_right_wheel"/>
         <xacro:inertial_wheel/>
     </link>
@@ -117,3 +119,4 @@
         <mimic joint="virtual_rear_wheel_joint" multiplier="1.0" offset="0.0"/>
     </joint>
+    </xacro:macro>
 </robot>

File: hunter_description/description/ros2_control.xacro (robot description, xacro)
@@ -1,10 +1,8 @@
 <?xml version="1.0"?>
 <robot xmlns:xacro="http://www.ros.org/wiki/xacro">
-  <xacro:macro name="carlikebot_ros2_control" params="name">
+  <xacro:macro name="hunter_ros2_control" params="name">
     <ros2_control name="${name}" type="system">
       <hardware>
         <plugin>hunter_description/CarlikeBotSystemHardware</plugin>
-        <param name="param_hw_start_duration_sec">0</param>
-        <param name="param_hw_stop_duration_sec">3.0</param>
       </hardware>
       <joint name="virtual_front_wheel_joint">

Commit message: adding Friction coefficient

File: hunter_description/description/meshes.xacro (robot description, xacro)
@@ -26,3 +26,12 @@
     </visual>
   </xacro:macro>
+  <xacro:macro name="gazebo_friction" params="reference">
+    <gazebo reference="${reference}">
+      <mu1 value="1.0"/>
+      <mu2 value="0.5"/>
+      <kp value="10000000.0" />
+      <kd value="1.0" />
+      <fdir1 value="1 0 0"/>
+    </gazebo>
+  </xacro:macro>
 </robot>

File: hunter_description/description/robot_core.xacro (robot description, xacro)
@@ -32,4 +32,5 @@
     <limit effort="10.0" velocity="10.0"/>
   </joint>
+  <xacro:gazebo_friction reference="rear_left_wheel"/>
   <link name="rear_right_wheel">
     <xacro:mesh name="rear_right_wheel"/>
@@ -45,4 +46,5 @@
     <mimic joint="rear_left_wheel_joint" multiplier="1.0" offset="0.0"/>
   </joint>
+  <xacro:gazebo_friction reference="rear_right_wheel"/>
   <link name="front_left_steering_link">
     <xacro:virtual/>
