Commit message: change wheel type

File: hunter_description/description/robot_core_real_hack.xacro (robot description, xacro)
@@ -24,5 +24,5 @@
     <xacro:inertial_wheel/>
   </link>
-  <joint name="rear_left_wheel_joint" type="fixed">
+  <joint name="rear_left_wheel_joint" type="continuous">
     <parent link="chassis"/>
     <child link="rear_left_wheel"/>
@@ -37,5 +37,5 @@
     <xacro:inertial_wheel/>
   </link>
-  <joint name="rear_right_wheel_joint" type="fixed">
+  <joint name="rear_right_wheel_joint" type="continuous">
     <parent link="chassis"/>
     <child link="rear_right_wheel"/>
@@ -51,5 +51,5 @@
     <xacro:inertial_steering_link/>
   </link>
-  <joint name="front_left_steering_joint" type="fixed">
+  <joint name="front_left_steering_joint" type="revolute">
     <parent link="chassis"/>
     <child link="front_left_steering_link"/>
@@ -63,9 +63,10 @@
     <xacro:inertial_wheel/>
   </link>
-  <joint name="front_left_wheel_joint" type="fixed">
+  <joint name="front_left_wheel_joint" type="continuous">
     <parent link="front_left_steering_link"/>
     <child link="front_left_wheel"/>
     <origin xyz="0 0 0" rpy="0 0 0" />
     <axis   xyz="0 0 -1" />
+    <mimic joint="rear_left_wheel_joint" multiplier="1.0" offset="0.0"/>
   </joint>
   <link name="front_right_steering_link">
@@ -73,5 +74,5 @@
     <xacro:inertial_steering_link/>
   </link>
-  <joint name="front_right_steering_joint" type="fixed">
+  <joint name="front_right_steering_joint" type="revolute">
     <parent link="chassis"/>
     <child link="front_right_steering_link"/>
@@ -86,9 +87,10 @@
     <xacro:inertial_wheel/>
   </link>
-  <joint name="front_right_wheel_joint" type="fixed">
+  <joint name="front_right_wheel_joint" type="continuous">
     <parent link="front_right_steering_link"/>
     <child link="front_right_wheel"/>
     <origin xyz="0 0 0" rpy="0 0 0" />
     <axis   xyz="0 0 -1" />
+    <mimic joint="rear_left_wheel_joint" multiplier="1.0" offset="0.0"/>
   </joint>
 </robot>
