Commit message: fix robot urdf and add steering joints

File: hunter_description/description/robot_core.xacro (robot description, xacro)
@@ -1,47 +1,187 @@
 <?xml version="1.0"?>
-<robot xmlns:xacro="http://www.ros.org/wiki/xacro" >
-<xacro:macro name="dogbot" params="prefix">
-    <xacro:property name="chassis_xyz" value="-0.016 -0.01 0.1025"/>
-    <!-- BASE LINK -->
-    <link name="base_link">
-    </link>
-    <!-- CHASSIS LINK -->
+<robot xmlns:xacro="http://www.ros.org/wiki/xacro" name="robot" >
+    <!-- <xacro:macro name="hunter_2" params="prefix"> -->
+    <!-- REF: https://youtu.be/BcjHyhV0kIs?si=dUpg7IF-kHSUgB-w -->
+    <!-- Robot website: https://robosavvy.co.uk/agilex-hunter-2b.html -->
+    <!-- Include the inertial values from the following -->
+    <xacro:include filename="inertial_macros.xacro"/>
+    <!-- BASE LINK ================================================================== -->
+    <link name="base_link"/>
+    <!-- CHASSIS JOINT & LINK ======================================================= -->
     <joint name="chassis_joint" type="fixed">
         <parent link="base_link"/>
         <child link="chassis"/>
+        <origin xyz="0 0 0.26" rpy="0 0 0" />
+    </joint>
+    <link name="chassis">
+        <visual>
+            <origin xyz="0 0 0" rpy="0 0 0"/>
+            <geometry>
+                <mesh filename="file://$(find hunter_description)/meshes/chassis.dae" />
+            </geometry>
+        </visual>
+        <collision>
+            <origin xyz="0 0 0" rpy="0 0 0"/>
+            <geometry>
+                <mesh filename="file://$(find hunter_description)/meshes/chassis.dae" />
+            </geometry>
+        </collision>
+        <xacro:inertial_chassis/>
+    </link>
+    <!-- ============================================================================ -->
+    <!-- REAR LEFT WHEEL JOINT & LINK -->
+    <joint name="rear_left_wheel_joint" type="continuous">
+        <parent link="chassis"/>
+        <child link="rear_left_wheel"/>
+        <origin xyz="-0.28 0.29249 -0.19558" rpy="${pi/2} 0 0" />
+        <axis   xyz="0 0 -1" />
+        <dynamics damping="0.0" friction="15"/>    </joint>
+    <link name="rear_left_wheel">
+        <visual>
+            <origin xyz="0 0 0" rpy="0 0 0" />
+            <geometry>
+                <mesh filename="file://$(find hunter_description)/meshes/rear_left_wheel.dae" />
+            </geometry>
+        </visual>
+        <collision>
+            <origin xyz="0 0 0" rpy="0 0 0" />
+            <geometry>
+                <mesh filename="file://$(find hunter_description)/meshes/rear_left_wheel.dae" />
+            </geometry>
+        </collision>
+        <xacro:inertial_wheel/>
+    </link>
+    <!-- =========================================================================-0.19558=== -->
+    <!-- REAR RIGHT WHEEL JOINT & LINK -->
+    <joint name="rear_right_wheel_joint" type="continuous">
+        <parent link="chassis"/>
+        <child link="rear_right_wheel"/>
+        <origin xyz="-0.28018 -0.29251 -0.19558" rpy="${pi/2} 0 0" />
+        <axis xyz="0.0 0.0 -1.0"/>
+        <dynamics damping="0.0" friction="15"/>
+    </joint>
+    <link name="rear_right_wheel">
+        <visual>
+            <origin xyz="0 0 0" rpy="0 0 0" />
+            <geometry>
+                <mesh filename="file://$(find hunter_description)/meshes/rear_right_wheel.dae" />
+            </geometry>
+        </visual>
+        <collision>
+            <origin xyz="0 0 0" rpy="0 0 0" />
+            <geometry>
+                <mesh filename="file://$(find hunter_description)/meshes/rear_right_wheel.dae" />
+            </geometry>
+        </collision>
+        <xacro:inertial_wheel/>
+    </link>
+    <!-- ============================================================================ -->
+    <!-- FRONT STEER LEFT WHEEL JOINT & LINK -->
+    <joint name="front_steer_left_wheel_joint" type="revolute">
+        <parent link="chassis"/>
+        <child link="front_steer_left_wheel"/>
+        <origin xyz="0.37142 0.29199 -0.1955" rpy="${pi/2} 0 0" />
+        <axis   xyz="0 1 0" />
+        <limit  lower="-0.69"  upper="0.69"  effort="0"  velocity="0" />
+    </joint>
+    <link name="front_steer_left_wheel">
+        <visual>
+            <origin xyz="0 0 0" rpy="0 0 0" />
+            <geometry>
+                <cylinder length="0.001" radius="0.005"/>
+            </geometry>
+            <material
+                name="">
+                <color rgba="0.79216 0.81961 0.93333 1" />
+            </material>
+        </visual>
+        <collision>
+            <origin xyz="0 0 0" rpy="0 0 0" />
+            <geometry>
+                <cylinder length="0.001" radius="0.005"/>
+            </geometry>
+        </collision>
+        <inertial>
+            <origin xyz="-0.012614 1.8116E-05 0.0023132" rpy="0 0 0" />
+            <mass value="0.8526" />
+            <inertia
+                ixx="0.063827"
+                ixy="0"
+                ixz="0"
+                iyy="0.063827"
+                iyz="0"
+                izz="0.11091" />
+        </inertial>
+    </link>
+    <!-- ============================================================================ -->
+    <!-- FRONT LEFT WHEEL JOINT & LINK -->
+    <joint name="front_left_wheel_joint" type="continuous">
+        <parent link="front_steer_left_wheel"/>
+        <child link="front_left_wheel"/>
         <origin xyz="0 0 0" rpy="0 0 0" />
-    </joint>
-    <link name="chassis">
-        <visual>
-            <origin xyz="${chassis_xyz}" rpy="0 0 0"/>
-            <geometry>
-                <mesh filename="file://$(find hunter_description)/meshes/chassis.dae" />
-            </geometry>
-            <material name="chassis">
-                <color rgba="0.752941176470588 0.752941176470588 0.752941176470588 1" />
+        <axis   xyz="0 0 -1" />
+        <dynamics damping="0.0" friction="15"/>
+    </joint>
+    <link name="front_left_wheel">
+        <visual>
+            <origin xyz="0 0 0" rpy="0 0 0" />
+            <geometry>
+                <mesh filename="file://$(find hunter_description)/meshes/front_left_wheel.dae" />
+            </geometry>
+        </visual>
+        <collision>
+            <origin xyz="0 0 0" rpy="0 0 0" />
+            <geometry>
+                <mesh filename="file://$(find hunter_description)/meshes/front_left_wheel.dae" />
+            </geometry>
+        </collision>
+        <xacro:inertial_wheel/>
+    </link>
+    <!-- ============================================================================ -->
+    <!-- FRONT STEER RIGHT WHEEL JOINT & LINK -->
+    <joint name="front_steer_right_wheel_joint" type="revolute">
+        <parent link="chassis"/>
+        <child link="front_steer_right_wheel"/>
+        <origin xyz="0.37142 -0.29201 -0.1955" rpy="${pi/2} 0 0" />
+        <axis   xyz="0 1 0" />
+        <limit  lower="-0.69"  upper="0.69"  effort="0"  velocity="0" />
+    </joint>
+    <link name="front_steer_right_wheel">
+        <visual>
+            <origin xyz="0 0 0" rpy="0 0 0" />
+            <geometry>
+                <cylinder length="0.001" radius="0.005"/>
+            </geometry>
+            <material
+                name="">
+                <color rgba="0.79216 0.81961 0.93333 1" />
             </material>
         </visual>
         <collision>
-            <origin xyz="${chassis_xyz}" rpy="0 0 0"/>
-            <geometry>
-                <mesh filename="file://$(find hunter_description)/meshes/chassis.dae" />
+            <origin xyz="0 0 0" rpy="0 0 0" />
+            <geometry>
+                <cylinder length="0.001" radius="0.005"/>
             </geometry>
         </collision>
         <inertial>
-            <origin xyz="${chassis_xyz}" rpy="0 0 0"/>
-            <mass value="24.7" />
-            <inertia ixx="0.123215829336501" ixy="-2.51201031615063E-06" ixz="0.00480100638469038" iyy="0.219144715482931" iyz="-1.0329581476775E-0" izz="0.313606030126045" />
+            <origin xyz="-8.9374E-08 1.0997E-07 0.0095958" rpy="0 0 0" />
+            <mass value="0.8526" />
+            <inertia
+                ixx="0.063827"
+                ixy="0"
+                ixz="0"
+                iyy="0.063827"
+                iyz="0"
+                izz="0.11091" />
         </inertial>
     </link>
-    <gazebo reference="chassis">
-        <material>Gazebo/Grey</material>
-    </gazebo>
-    <!-- FRONT RIGHT WHEEL LINK -->
+    <!-- ============================================================================ -->
+    <!-- FRONT RIGHT WHEEL JOINT & LINK -->
     <joint name="front_right_wheel_joint" type="continuous">
-        <parent link="base_link"/>
+        <parent link="front_steer_right_wheel"/>
         <child link="front_right_wheel"/>
-        <origin xyz="0.215 0.263 0.096" rpy="${-pi/2} 0 0" />
-        <axis xyz="0.0 0.0 1.0"/>
-        <!-- <dynamics damping="0.02" friction="0.02" /> -->
+        <origin xyz="0 0 0" rpy="0 0 0" />
+        <axis xyz="0 0 -1" />
+        <dynamics damping="0.0" friction="15"/>
     </joint>
     <link name="front_right_wheel">
@@ -49,126 +189,15 @@
             <origin xyz="0 0 0" rpy="0 0 0" />
             <geometry>
-                <mesh filename="file://$(find hunter_description)/meshes/wheel.dae" />
-            </geometry>
-            <material name="wheel">
-                <color rgba="0.0 0.0 0.0 1" />
-            </material>
-        </visual>
-        <collision>
-            <origin xyz="0 0 -0.03" rpy="0 0 0" />
-            <geometry>
-                <mesh filename="file://$(find hunter_description)/meshes/wheel.dae" />
-            </geometry>
-        </collision>
-        <inertial>
-            <origin xyz="0.00027498198567355 3.24801296969213E-11 -0.0163540222836661" rpy="0 0 0" />
-            <mass value="3.149" />
-            <inertia ixx="0.0222" ixy="0.0" ixz="0.0" iyy="0.0222" iyz="0.0" izz="0.0378075" />
-        </inertial>
-    </link>
-    <gazebo reference="front_right_wheel">
-        <material>Gazebo/DarkGrey</material>
-    </gazebo>
-    <!-- FRONT LEFT WHEEL LINK -->
-    <joint name="front_left_wheel_joint" type="continuous">
-        <parent link="base_link"/>
-        <child link="front_left_wheel"/>
-        <origin xyz="0.34058 0.24619 -0.1535" rpy="${-pi/2} 0 0" />
-        <axis xyz="0.0 0.0 1.0"/>
-        <!-- <dynamics damping="0.02" friction="0.02" /> -->
-    </joint>
-    <link name="front_left_wheel">
-        <visual>
-            <origin xyz="0 0 0" rpy="0 0 0" />
-            <geometry>
-                <mesh filename="file://$(find hunter_description)/meshes/wheel.dae" />
-            </geometry>
-            <material name="wheel">
-                <color rgba="0.0 0.0 0.0 1" />
-            </material>
-        </visual>
-        <collision>
-            <origin xyz="0 0 -0.03" rpy="0 0 0" />
-            <geometry>
-                <mesh filename="file://$(find hunter_description)/meshes/wheel.dae" />
-            </geometry>
-        </collision>
-        <inertial>
-            <origin xyz="-3.5837499634539E-10 4.97346158701006E-09 -0.016356334080185" rpy="0 0 0" />
-            <mass value="3.149" />
-            <inertia ixx="0.0222" ixy="0.0" ixz="0.0" iyy="0.0222" iyz="0.0" izz="0.0378075" />
-        </inertial>
-    </link>
-    <gazebo reference="front_left_wheel">
-        <material>Gazebo/DarkGrey</material>
-    </gazebo>
-    <!-- BACK RIGHT WHEEL LINK -->
-    <joint name="back_right_wheel_joint" type="continuous">
-        <parent link="base_link"/>
-        <child link="back_right_wheel"/>
-        <origin xyz="-0.2078 -0.252 -0.158" rpy="${-pi/2} 0 0" />
-        <axis xyz="0.0 0.0 1.0"/>
-        <!-- <dynamics damping="0.02" friction="0.02" /> -->
-        <!-- <mimic joint="front_right_wheel_joint" multiplier="1" offset="0" /> -->
-    </joint>
-    <link name="back_right_wheel">
-        <visual>
-            <origin xyz="0 0 -0.03" rpy="0 0 0" />
-            <geometry>
-                <mesh filename="file://$(find hunter_description)/meshes/wheel.dae" />
-            </geometry>
-            <material name="wheel">
-                <color rgba="0.0 0.0 0.0 1" />
-            </material>
-        </visual>
-        <collision>
-            <origin xyz="0 0 -0.03" rpy="0 0 0" />
-            <geometry>
-                <mesh filename="file://$(find hunter_description)/meshes/wheel.dae" />
-            </geometry>
-        </collision>
-        <inertial>
-            <origin xyz="0 0 -0.03" rpy="0 0 0" />
-            <mass value="1" />
-            <inertia ixx="0.0222" ixy="0.0" ixz="0.0" iyy="0.0222" iyz="0.0" izz="0.037807" />
-        </inertial>
-    </link>
-    <gazebo reference="back_right_wheel">
-        <material>Gazebo/DarkGrey</material>
-    </gazebo>
-    <!-- BACK LEFT WHEEL LINK -->
-    <joint name="back_left_wheel_joint" type="continuous">
-        <parent link="base_link"/>
-        <child link="back_left_wheel"/>
-        <origin xyz="-0.2078 0.252 -0.158" rpy="${-pi/2} 0 0" />
-        <axis xyz="0.0 0.0 1.0"/>
-        <!-- <dynamics damping="0.02" friction="0.02" /> -->
-        <!-- <mimic joint="front_left_wheel_joint" multiplier="1" offset="0" /> -->
-    </joint>
-    <link name="back_left_wheel">
-        <visual>
-            <origin xyz="0 0 -0.03" rpy="0 0 0" />
-            <geometry>
-                <mesh filename="file://$(find hunter_description)/meshes/wheel.dae" />
-            </geometry>
-            <material name="wheel">
-                <color rgba="0.0 0.0 0.0 1" />
-            </material>
-        </visual>
-        <collision>
-            <origin xyz="0 0 -0.03" rpy="0 0 0" />
-            <geometry>
-                <mesh filename="file://$(find hunter_description)/meshes/wheel.dae" />
-            </geometry>
-        </collision>
-        <inertial>
-            <origin xyz="0 0 -0.03" rpy="0 0 0" />
-            <mass value="3.149" />
-            <inertia ixx="0.0222" ixy="0.0" ixz="0.0" iyy="0.0222" iyz="0.0" izz="0.0378075" />
-        </inertial>
-    </link>
-    <gazebo reference="back_left_wheel">
-        <material>Gazebo/DarkGrey</material>
-    </gazebo>
-    </xacro:macro>
+                <mesh filename="file://$(find hunter_description)/meshes/front_right_wheel.dae" />
+            </geometry>
+        </visual>
+        <collision>
+            <origin xyz="0 0 0" rpy="0 0 0" />
+            <geometry>
+                <mesh filename="file://$(find hunter_description)/meshes/front_right_wheel.dae" />
+            </geometry>
+        </collision>
+        <xacro:inertial_wheel/>
+    </link>
+    <!-- </xacro:macro> -->
 </robot>
