Commit message: simplify hunter urdf model

File: hunter_description/description/robot_core.xacro (robot description, xacro)
@@ -28,13 +28,26 @@
         <xacro:inertial_chassis/>
     </link>
-    <!-- ============================================================================ -->
+    <!-- REAR WHEELS ================================================================ -->
+    <!-- VIRTUAL REAR WHEEL -->
+    <link name="virtual_rear_wheel">
+        <visual>
+            <origin xyz="0 0 0" rpy="0 0 0"/>
+            <geometry>
+                <cylinder length="0.01" radius="0.165"/>
+            </geometry>
+            <material name="invisible">
+                <color rgba="0.0 0.0 0.0 0.0"/>
+            </material>
+        </visual>
+    </link>
+    <joint name="virtual_rear_wheel_joint" type="continuous">
+        <parent link="chassis"/>
+        <child link="virtual_rear_wheel"/>
+        <origin xyz="-0.28 0.0 -0.19558" rpy="${pi/2} 0 0"/>
+        <axis xyz="0 0 -1"/>
+        <limit effort="10.0" velocity="10.0"/>
+        <dynamics damping="0.2"/>
+    </joint>
     <!-- REAR LEFT WHEEL JOINT & LINK -->
-    <joint name="rear_left_wheel_joint" type="continuous">
-        <parent link="chassis"/>
-        <child link="rear_left_wheel"/>
-        <origin xyz="-0.28 0.29249 -0.19558" rpy="${pi/2} 0 0" />
-        <axis   xyz="0 0 -1" />
-        <dynamics damping="0.0" friction="15"/>
-    </joint>
     <link name="rear_left_wheel">
         <visual>
@@ -52,13 +65,14 @@
         <xacro:inertial_wheel/>
     </link>
-    <!-- =========================================================================-0.19558=== -->
+    <joint name="rear_left_wheel_joint" type="continuous">
+        <parent link="chassis"/>
+        <child link="rear_left_wheel"/>
+        <origin xyz="-0.28 0.29249 -0.19558" rpy="${pi/2} 0 0" />
+        <axis   xyz="0 0 -1" />
+        <dynamics damping="0.2" friction="15"/>
+        <limit effort="10.0" velocity="10.0"/>
+        <mimic joint="virtual_rear_wheel_joint" multiplier="1.0" offset="0.0"/>
+    </joint>
     <!-- REAR RIGHT WHEEL JOINT & LINK -->
-    <joint name="rear_right_wheel_joint" type="continuous">
-        <parent link="chassis"/>
-        <child link="rear_right_wheel"/>
-        <origin xyz="-0.28018 -0.29251 -0.19558" rpy="${pi/2} 0 0" />
-        <axis xyz="0.0 0.0 -1.0"/>
-        <dynamics damping="0.0" friction="15"/>
-    </joint>
     <link name="rear_right_wheel">
         <visual>
@@ -76,84 +90,35 @@
         <xacro:inertial_wheel/>
     </link>
+    <joint name="rear_right_wheel_joint" type="continuous">
+        <parent link="chassis"/>
+        <child link="rear_right_wheel"/>
+        <origin xyz="-0.28018 -0.29251 -0.19558" rpy="${pi/2} 0 0" />
+        <axis xyz="0.0 0.0 -1.0"/>
+        <dynamics damping="0.2" friction="15"/>
+        <limit effort="10.0" velocity="10.0"/>
+        <mimic joint="virtual_rear_wheel_joint" multiplier="1.0" offset="0.0"/>
+    </joint>
     <!-- ============================================================================ -->
-    <!-- FRONT STEER JOINT & LINK -->
-    <joint name="front_steer_joint" type="fixed">
-        <origin xyz="0.44792 -1.1431E-05 -0.121" rpy="0 0 0" />
-        <parent link="chassis" />
-        <child  link="front_steer" />
-        <axis   xyz="0 0 0" />
-    </joint>
-    <link name="front_steer">
+    <!-- VIRTUAL FRONT WHEEL -->
+    <link name="virtual_front_wheel">
         <visual>
-            <origin xyz="0 0 0" rpy="0 0 0" />
+            <origin xyz="0 0 0" rpy="0 0 0"/>
             <geometry>
-                <mesh filename="file://$(find hunter_description)/meshes/front_steer_link.STL" />
+                <cylinder length="0.01" radius="0.165"/>
             </geometry>
-        </visual>
-        <collision>
-            <origin xyz="0 0 0" rpy="0 0 0" />
-            <geometry>
-                <mesh filename="file://$(find hunter_description)/meshes/front_steer_link.STL" />
-            </geometry>
-        </collision>
-        <inertial>
-            <origin xyz="0.049836 8.1046E-15 0.017912" rpy="0 0 0" />
-            <mass value="0.0049179" />
-            <inertia
-                ixx="1.6846E-07"
-                ixy="7.6396E-23"
-                ixz="-1.0974E-08"
-                iyy="7.549E-07"
-                iyz="-1.8957E-22"
-                izz="7.334E-07" />
-        </inertial>
-    </link>
-    <!-- ============================================================================ -->
-    <!-- FRONT STEER LEFT WHEEL JOINT & LINK -->
-    <joint name="front_left_steer_joint" type="revolute">
-        <parent link="chassis"/>
-        <child link="front_steer_left_wheel"/>
-        <origin xyz="0.37142 0.29199 -0.1955" rpy="${pi/2} 0 0" />
-        <axis   xyz="0 1 0" />
-        <limit  lower="-0.69"  upper="0.69"  effort="0"  velocity="0" />
-    </joint>
-    <link name="front_steer_left_wheel">
-        <visual>
-            <origin xyz="0 0 0" rpy="0 0 0" />
-            <geometry>
-                <cylinder length="0.001" radius="0.005"/>
-            </geometry>
-            <material
-                name="">
-                <color rgba="0.79216 0.81961 0.93333 1" />
+            <material name="invisible">
+                <color rgba="0.0 0.0 0.0 0.0"/>
             </material>
         </visual>
-        <collision>
-            <origin xyz="0 0 0" rpy="0 0 0" />
-            <geometry>
-                <cylinder length="0.001" radius="0.005"/>
-            </geometry>
-        </collision>
-        <inertial>
-            <origin xyz="-0.012614 1.8116E-05 0.0023132" rpy="0 0 0" />
-            <mass value="0.8526" />
-            <inertia
-                ixx="0.063827"
-                ixy="0"
-                ixz="0"
-                iyy="0.063827"
-                iyz="0"
-                izz="0.11091" />
-        </inertial>
     </link>
-    <!-- ============================================================================ -->
+    <joint name="virtual_front_wheel_joint" type="revolute">
+        <parent link="chassis"/>
+        <child link="virtual_front_wheel"/>
+        <origin xyz="0.37142 0 -0.1955" rpy="${pi/2} 0 0" />
+        <axis   xyz="0 1 0" />
+        <limit  lower="-0.69"  upper="0.69"  effort="10.0"  velocity="0" />
+        <dynamics damping="0.2"/>
+    </joint>
     <!-- FRONT LEFT WHEEL JOINT & LINK -->
-    <joint name="front_left_wheel_joint" type="continuous">
-        <parent link="front_steer_left_wheel"/>
-        <child link="front_left_wheel"/>
-        <origin xyz="0 0 0" rpy="0 0 0" />
-        <axis   xyz="0 0 -1" />
-        <dynamics damping="0.0" friction="15"/>
-    </joint>
     <link name="front_left_wheel">
         <visual>
@@ -171,51 +136,14 @@
         <xacro:inertial_wheel/>
     </link>
-    <!-- ============================================================================ -->
-    <!-- FRONT STEER RIGHT WHEEL JOINT & LINK -->
-    <joint name="front_right_steer_joint" type="revolute">
+    <joint name="front_left_wheel_joint" type="revolute">
         <parent link="chassis"/>
-        <child link="front_steer_right_wheel"/>
-        <origin xyz="0.37142 -0.29201 -0.1955" rpy="${pi/2} 0 0" />
+        <child link="front_left_wheel"/>
+        <origin xyz="0.37142 0.29199 -0.1955" rpy="${pi/2} 0 0" />
         <axis   xyz="0 1 0" />
-        <limit  lower="-0.69"  upper="0.69"  effort="0"  velocity="0" />
+        <limit  lower="-0.69"  upper="0.69"  effort="10.0"  velocity="0" />
+        <dynamics damping="0.2"/>
+        <mimic joint="virtual_front_wheel_joint" multiplier="1.0" offset="0.0"/>
     </joint>
-    <link name="front_steer_right_wheel">
-        <visual>
-            <origin xyz="0 0 0" rpy="0 0 0" />
-            <geometry>
-                <cylinder length="0.001" radius="0.005"/>
-            </geometry>
-            <material
-                name="">
-                <color rgba="0.79216 0.81961 0.93333 1" />
-            </material>
-        </visual>
-        <collision>
-            <origin xyz="0 0 0" rpy="0 0 0" />
-            <geometry>
-                <cylinder length="0.001" radius="0.005"/>
-            </geometry>
-        </collision>
-        <inertial>
-            <origin xyz="-8.9374E-08 1.0997E-07 0.0095958" rpy="0 0 0" />
-            <mass value="0.8526" />
-            <inertia
-                ixx="0.063827"
-                ixy="0"
-                ixz="0"
-                iyy="0.063827"
-                iyz="0"
-                izz="0.11091" />
-        </inertial>
-    </link>
-    <!-- ============================================================================ -->
     <!-- FRONT RIGHT WHEEL JOINT & LINK -->
-    <joint name="front_right_wheel_joint" type="continuous">
-        <parent link="front_steer_right_wheel"/>
-        <child link="front_right_wheel"/>
-        <origin xyz="0 0 0" rpy="0 0 0" />
-        <axis xyz="0 0 -1" />
-        <dynamics damping="0.0" friction="15"/>
-    </joint>
     <link name="front_right_wheel">
         <visual>
@@ -233,3 +161,12 @@
         <xacro:inertial_wheel/>
     </link>
+    <joint name="front_right_wheel_joint" type="revolute">
+        <parent link="chassis"/>
+        <child link="front_right_wheel"/>
+        <origin xyz="0.37142 -0.29199 -0.1955" rpy="${pi/2} 0 0" />
+        <axis   xyz="0 1 0" />
+        <limit  lower="-0.69"  upper="0.69"  effort="10.0"  velocity="0" />
+        <dynamics damping="0.2"/>
+        <mimic joint="virtual_front_wheel_joint" multiplier="1.0" offset="0.0"/>
+    </joint>
 </robot>

Commit message: added two new links for the wheels and simplify the controller

File: hunter_description/description/robot_core.xacro (robot description, xacro)
@@ -35,15 +35,5 @@
     <!-- REAR WHEELS ================================================================ -->
     <!-- VIRTUAL REAR WHEEL -->
-    <link name="virtual_rear_wheel">
-        <visual>
-            <origin xyz="0 0 0" rpy="0 0 0"/>
-            <geometry>
-                <cylinder length="0.01" radius="0.01"/>
-            </geometry>
-            <material name="invisible">
-                <color rgba="0.0 0.0 0.0 0.0"/>
-            </material>
-        </visual>
-    </link>
+    <link name="virtual_rear_wheel"/>
     <joint name="virtual_rear_wheel_joint" type="continuous">
         <parent link="chassis"/>
@@ -106,15 +96,5 @@
     <!-- ============================================================================ -->
     <!-- VIRTUAL FRONT WHEEL -->
-    <link name="virtual_front_wheel">
-        <visual>
-            <origin xyz="0 0 0" rpy="0 0 0"/>
-            <geometry>
-                <cylinder length="0.01" radius="0.01"/>
-            </geometry>
-            <material name="invisible">
-                <color rgba="0.0 0.0 0.0 0.0"/>
-            </material>
-        </visual>
-    </link>
+    <link name="virtual_front_wheel"/>
     <joint name="virtual_front_wheel_joint" type="revolute">
         <parent link="chassis"/>
@@ -126,5 +106,15 @@
     </joint>
     <!-- FRONT LEFT WHEEL JOINT & LINK -->
-    <link name="front_left_wheel">
+    <link name="front_left_wheel"/>
+    <joint name="front_left_wheel_joint" type="revolute">
+        <parent link="chassis"/>
+        <child link="front_left_wheel"/>
+        <origin xyz="${x_base_to_front} ${y_base_to_wheel} ${z_base_to_wheel}" rpy="${pi/2} 0 0" />
+        <axis   xyz="0 1 0" />
+        <limit  lower="-0.69"  upper="0.69"  effort="10.0"  velocity="0" />
+        <dynamics damping="0.2"/>
+        <mimic joint="virtual_front_wheel_joint" multiplier="1.0" offset="0.0"/>
+    </joint>
+    <link name="front_left_wheel_cont">
         <visual>
             <origin xyz="0 0 0" rpy="0 0 0" />
@@ -141,8 +131,17 @@
         <xacro:inertial_wheel/>
     </link>
-    <joint name="front_left_wheel_joint" type="revolute">
+    <joint name="front_left_wheel_cont_joint" type="continuous">
+        <parent link="front_left_wheel"/>
+        <child link="front_left_wheel_cont"/>
+        <origin xyz="0 0 0" rpy="0 0 0" />
+        <axis   xyz="0 0 -1" />
+        <mimic joint="virtual_rear_wheel_joint" multiplier="1.0" offset="0.0"/>
+    </joint>
+    <!-- FRONT RIGHT WHEEL JOINT & LINK -->
+    <link name="front_right_wheel"/>
+    <joint name="front_right_wheel_joint" type="revolute">
         <parent link="chassis"/>
-        <child link="front_left_wheel"/>
-        <origin xyz="${x_base_to_front} ${y_base_to_wheel} ${z_base_to_wheel}" rpy="${pi/2} 0 0" />
+        <child link="front_right_wheel"/>
+        <origin xyz="${x_base_to_front}  -${y_base_to_wheel} ${z_base_to_wheel}" rpy="${pi/2} 0 0" />
         <axis   xyz="0 1 0" />
         <limit  lower="-0.69"  upper="0.69"  effort="10.0"  velocity="0" />
@@ -150,6 +149,5 @@
         <mimic joint="virtual_front_wheel_joint" multiplier="1.0" offset="0.0"/>
     </joint>
-    <!-- FRONT RIGHT WHEEL JOINT & LINK -->
-    <link name="front_right_wheel">
+    <link name="front_right_wheel_cont">
         <visual>
             <origin xyz="0 0 0" rpy="0 0 0" />
@@ -166,12 +164,10 @@
         <xacro:inertial_wheel/>
     </link>
-    <joint name="front_right_wheel_joint" type="revolute">
-        <parent link="chassis"/>
-        <child link="front_right_wheel"/>
-        <origin xyz="${x_base_to_front}  -${y_base_to_wheel} ${z_base_to_wheel}" rpy="${pi/2} 0 0" />
-        <axis   xyz="0 1 0" />
-        <limit  lower="-0.69"  upper="0.69"  effort="10.0"  velocity="0" />
-        <dynamics damping="0.2"/>
-        <mimic joint="virtual_front_wheel_joint" multiplier="1.0" offset="0.0"/>
+    <joint name="front_right_wheel_cont_joint" type="continuous">
+        <parent link="front_right_wheel"/>
+        <child link="front_right_wheel_cont"/>
+        <origin xyz="0 0 0" rpy="0 0 0" />
+        <axis   xyz="0 0 -1" />
+        <mimic joint="virtual_rear_wheel_joint" multiplier="1.0" offset="0.0"/>
     </joint>
 </robot>

Commit message: move meshes into new xacro

File: hunter_description/description/robot_core.xacro (robot description, xacro)
@@ -5,4 +5,5 @@
     <!-- Include the inertial values from the following -->
     <xacro:include filename="inertial_macros.xacro"/>
+    <xacro:include filename="meshes.xacro"/>
     <!-- Constants for robot dimensions -->
     <xacro:property name="z_base_to_wheel" value="-0.19558" />
@@ -19,16 +20,5 @@
     </joint>
     <link name="chassis">
-        <visual>
-            <origin xyz="0 0 0" rpy="0 0 0"/>
-            <geometry>
-                <mesh filename="file://$(find hunter_description)/meshes/chassis.dae" />
-            </geometry>
-        </visual>
-        <collision>
-            <origin xyz="0 0 0" rpy="0 0 0"/>
-            <geometry>
-                <mesh filename="file://$(find hunter_description)/meshes/chassis.dae" />
-            </geometry>
-        </collision>
+        <xacro:chassis_mesh/>
         <xacro:inertial_chassis/>
     </link>
@@ -46,16 +36,5 @@
     <!-- REAR LEFT WHEEL JOINT & LINK -->
     <link name="rear_left_wheel">
-        <visual>
-            <origin xyz="0 0 0" rpy="0 0 0" />
-            <geometry>
-                <mesh filename="file://$(find hunter_description)/meshes/rear_left_wheel.dae" />
-            </geometry>
-        </visual>
-        <collision>
-            <origin xyz="0 0 0" rpy="0 0 0" />
-            <geometry>
-                <mesh filename="file://$(find hunter_description)/meshes/rear_left_wheel.dae" />
-            </geometry>
-        </collision>
+        <xacro:rear_left_wheel_mesh/>
         <xacro:inertial_wheel/>
     </link>
@@ -71,16 +50,5 @@
     <!-- REAR RIGHT WHEEL JOINT & LINK -->
     <link name="rear_right_wheel">
-        <visual>
-            <origin xyz="0 0 0" rpy="0 0 0" />
-            <geometry>
-                <mesh filename="file://$(find hunter_description)/meshes/rear_right_wheel.dae" />
-            </geometry>
-        </visual>
-        <collision>
-            <origin xyz="0 0 0" rpy="0 0 0" />
-            <geometry>
-                <mesh filename="file://$(find hunter_description)/meshes/rear_right_wheel.dae" />
-            </geometry>
-        </collision>
+        <xacro:rear_right_wheel_mesh/>
         <xacro:inertial_wheel/>
     </link>
@@ -117,16 +85,5 @@
     </joint>
     <link name="front_left_wheel_cont">
-        <visual>
-            <origin xyz="0 0 0" rpy="0 0 0" />
-            <geometry>
-                <mesh filename="file://$(find hunter_description)/meshes/front_left_wheel.dae" />
-            </geometry>
-        </visual>
-        <collision>
-            <origin xyz="0 0 0" rpy="0 0 0" />
-            <geometry>
-                <mesh filename="file://$(find hunter_description)/meshes/front_left_wheel.dae" />
-            </geometry>
-        </collision>
+        <xacro:front_left_wheel_mesh/>
         <xacro:inertial_wheel/>
     </link>
@@ -150,16 +107,5 @@
     </joint>
     <link name="front_right_wheel_cont">
-        <visual>
-            <origin xyz="0 0 0" rpy="0 0 0" />
-            <geometry>
-                <mesh filename="file://$(find hunter_description)/meshes/front_right_wheel.dae" />
-            </geometry>
-        </visual>
-        <collision>
-            <origin xyz="0 0 0" rpy="0 0 0" />
-            <geometry>
-                <mesh filename="file://$(find hunter_description)/meshes/front_right_wheel.dae" />
-            </geometry>
-        </collision>
+        <xacro:front_right_wheel_mesh/>
         <xacro:inertial_wheel/>
     </link>

Commit message: add real ackermann controller and update dynamics parameters

File: hunter_description/description/robot_core.xacro (robot description, xacro)
@@ -44,5 +44,5 @@
     <dynamics damping="0.2" friction="15"/>
     <limit effort="10.0" velocity="10.0"/>
-    <mimic joint="rear_left_wheel_joint" multiplier="1.0" offset="0.0"/>
+    <!-- <mimic joint="rear_left_wheel_joint" multiplier="1.0" offset="0.0"/> -->
   </joint>
   <xacro:gazebo_friction reference="rear_right_wheel"/>
@@ -57,5 +57,5 @@
     <axis   xyz="0 1 0" />
     <limit  lower="-${max_steer_angle_central}"  upper="${max_steer_angle_central}"  effort="10.0"  velocity="1" />
-    <dynamics damping="0.2"/>
+    <dynamics damping="1.0"/>
   </joint>
   <link name="front_left_wheel">
@@ -79,6 +79,6 @@
     <axis   xyz="0 1 0" />
     <limit  lower="-${max_steer_angle_central}"  upper="${max_steer_angle_central}"  effort="10.0"  velocity="1" />
-    <dynamics damping="0.2"/>
-    <mimic joint="front_left_steering_joint" multiplier="1.0" offset="0.0"/>
+    <dynamics damping="1.0"/>
+    <!-- <mimic joint="front_left_steering_joint" multiplier="1.0" offset="0.0"/> -->
   </joint>
   <link name="front_right_wheel">

File: hunter_description/description/ros2_control.xacro (robot description, xacro)
@@ -10,6 +10,5 @@
     </joint>
     <joint name="front_right_steering_joint">
-      <param name="mimic">front_left_steering_joint</param>
-      <param name="multiplier">1</param>
+      <command_interface name="position"/>
       <state_interface name="position"/>
     </joint>
@@ -20,6 +19,5 @@
     </joint>
     <joint name="rear_right_wheel_joint">
-      <param name="mimic">rear_left_wheel_joint</param>
-      <param name="multiplier">1</param>
+      <command_interface name="velocity"/>
       <state_interface name="velocity"/>
       <state_interface name="position"/>
